Commit message: model by pkg

File: iri_wam_description/urdf/wam.urdf (robot description, URDF)
Before this commit: robot iri_wam, 10 links, 9 joints
Links:
- link iri_wam_link_1: geometry collision mesh filename=package://iri_wam_description/mesh/wam1_collision.stl scale=1.0 1.0 1.0; visual mesh filename=package://iri_wam_description/mesh/wam1.stl scale=1.0 1.0 1.0
- link iri_wam_link_2: geometry collision mesh filename=package://iri_wam_description/mesh/wam2_collision.stl scale=1.0 1.0 1.0; visual mesh filename=package://iri_wam_description/mesh/wam2.stl scale=1.0 1.0 1.0
- link iri_wam_link_3: geometry collision mesh filename=package://iri_wam_description/mesh/wam3_collision.stl scale=1.0 1.0 1.0; visual mesh filename=package://iri_wam_description/mesh/wam3.stl scale=1.0 1.0 1.0
- link iri_wam_link_4: geometry collision mesh filename=package://iri_wam_description/mesh/wam4_collision.stl scale=1.0 1.0 1.0; visual mesh filename=package://iri_wam_description/mesh/wam4.stl scale=1.0 1.0 1.0
- link iri_wam_link_5: geometry collision mesh filename=package://iri_wam_description/mesh/wam5_collision.stl scale=1.0 1.0 1.0; visual mesh filename=package://iri_wam_description/mesh/wam5.stl scale=1.0 1.0 1.0
- link iri_wam_link_6: geometry collision mesh filename=package://iri_wam_description/mesh/wam6_collision.stl scale=1.0 1.0 1.0; visual mesh filename=package://iri_wam_description/mesh/wam6.stl scale=1.0 1.0 1.0
- link iri_wam_link_7: geometry collision mesh filename=package://iri_wam_description/mesh/wam7_collision.stl scale=1.0 1.0 1.0; visual mesh filename=package://iri_wam_description/mesh/wam7.stl scale=1.0 1.0 1.0
- link iri_wam_link_base: geometry collision mesh filename=package://iri_wam_description/mesh/wambase_collision.stl scale=1.0 1.0 1.0; visual mesh filename=package://iri_wam_description/mesh/wambase.stl scale=1.0 1.0 1.0

File: iri_wam_description/urdf/wam_gazebo.urdf (robot description, URDF)
Before this commit: robot iri_wam, 11 links, 10 joints
Links:
- link iri_wam_link_1: geometry collision mesh filename=package://iri_wam_description/mesh/wam1_collision.stl scale=1.0 1.0 1.0; visual mesh filename=package://iri_wam_description/mesh/wam1.stl scale=1.0 1.0 1.0
- link iri_wam_link_2: geometry collision mesh filename=package://iri_wam_description/mesh/wam2_collision.stl scale=1.0 1.0 1.0; visual mesh filename=package://iri_wam_description/mesh/wam2.stl scale=1.0 1.0 1.0
- link iri_wam_link_3: geometry collision mesh filename=package://iri_wam_description/mesh/wam3_collision.stl scale=1.0 1.0 1.0; visual mesh filename=package://iri_wam_description/mesh/wam3.stl scale=1.0 1.0 1.0
- link iri_wam_link_4: geometry collision mesh filename=package://iri_wam_description/mesh/wam4_collision.stl scale=1.0 1.0 1.0; visual mesh filename=package://iri_wam_description/mesh/wam4.stl scale=1.0 1.0 1.0
- link iri_wam_link_5: geometry collision mesh filename=package://iri_wam_description/mesh/wam5_collision.stl scale=1.0 1.0 1.0; visual mesh filename=package://iri_wam_description/mesh/wam5.stl scale=1.0 1.0 1.0
- link iri_wam_link_6: geometry collision mesh filename=package://iri_wam_description/mesh/wam6_collision.stl scale=1.0 1.0 1.0; visual mesh filename=package://iri_wam_description/mesh/wam6.stl scale=1.0 1.0 1.0
- link iri_wam_link_7: geometry collision mesh filename=package://iri_wam_description/mesh/wam7_collision.stl scale=1.0 1.0 1.0; visual mesh filename=package://iri_wam_description/mesh/wam7.stl scale=1.0 1.0 1.0
- link iri_wam_link_base: geometry collision mesh filename=package://iri_wam_description/mesh/wambase_collision.stl scale=1.0 1.0 1.0; visual mesh filename=package://iri_wam_description/mesh/wambase.stl scale=1.0 1.0 1.0

File: iri_wam_description/xacro/iri_wam_1.urdf.xacro (robot description, xacro)
@@ -14,5 +14,5 @@
             <origin xyz="0.0 0.0 0.0" rpy="0 0 0" />
             <geometry name="${prefix}_link_1_visual">
-                <mesh filename="model://iri_wam_description/mesh/wam1.stl" scale="1.0 1.0 1.0" />
+                <mesh filename="package://iri_wam_description/mesh/wam1.stl" scale="1.0 1.0 1.0" />
             </geometry>
             <material name="Grey" >
@@ -23,5 +23,5 @@
             <origin xyz="0.0 0.0 0.0" rpy="0 0 0"/>
             <geometry name="${prefix}_link_1_collision">
-                <mesh filename="model://iri_wam_description/mesh/wam1_collision.stl" scale="1.0 1.0 1.0" />
+                <mesh filename="package://iri_wam_description/mesh/wam1_collision.stl" scale="1.0 1.0 1.0" />
 <!--                <box size="0.20 0.40 0.40"/> -->
             </geometry>

File: iri_wam_description/xacro/iri_wam_2.urdf.xacro (robot description, xacro)
@@ -14,5 +14,5 @@
             <origin xyz="0.0 0.0 0.0" rpy="0 0 0" />
             <geometry name="${prefix}_link_2_visual">
-                <mesh filename="model://iri_wam_description/mesh/wam2.stl" scale="1.0 1.0 1.0" />
+                <mesh filename="package://iri_wam_description/mesh/wam2.stl" scale="1.0 1.0 1.0" />
             </geometry>
             <material name="Grey" >
@@ -23,5 +23,5 @@
             <origin xyz="0.0 0.0 0.0" rpy="0 0 0"/>
             <geometry name="${prefix}_link_2_collision">
-                <mesh filename="model://iri_wam_description/mesh/wam2_collision.stl" scale="1.0 1.0 1.0" />
+                <mesh filename="package://iri_wam_description/mesh/wam2_collision.stl" scale="1.0 1.0 1.0" />
 <!--                <box size="0.10 0.10 0.10"/> -->
             </geometry>

File: iri_wam_description/xacro/iri_wam_3.urdf.xacro (robot description, xacro)
@@ -14,5 +14,5 @@
             <origin xyz="0.0 0.0 0.0" rpy="0 0 0" />
             <geometry name="${prefix}_link_3_visual">
-                <mesh filename="model://iri_wam_description/mesh/wam3.stl" scale="1.0 1.0 1.0" />
+                <mesh filename="package://iri_wam_description/mesh/wam3.stl" scale="1.0 1.0 1.0" />
             </geometry>
             <material name="Grey" >
@@ -23,5 +23,5 @@
             <origin xyz="0.0 0.0 0.0" rpy="0 0 0"/>
             <geometry name="${prefix}_link_3_collision">
-                <mesh filename="model://iri_wam_description/mesh/wam3_collision.stl" scale="1.0 1.0 1.0" />
+                <mesh filename="package://iri_wam_description/mesh/wam3_collision.stl" scale="1.0 1.0 1.0" />
 <!--                <cylinder length="0.6" radius="0.02"/> -->
             </geometry>

File: iri_wam_description/xacro/iri_wam_4.urdf.xacro (robot description, xacro)
@@ -14,5 +14,5 @@
             <origin xyz="0.0 0.0 0.0" rpy="0 0 0" />
             <geometry name="${prefix}_link_4_visual">
-                <mesh filename="model://iri_wam_description/mesh/wam4.stl" scale="1.0 1.0 1.0" />
+                <mesh filename="package://iri_wam_description/mesh/wam4.stl" scale="1.0 1.0 1.0" />
             </geometry>
             <material name="Grey" >
@@ -23,5 +23,5 @@
             <origin xyz="0.0 0.0 0.0" rpy="0 0 0"/>
             <geometry name="${prefix}_link_4_collision">
-                <mesh filename="model://iri_wam_description/mesh/wam4_collision.stl" scale="1.0 1.0 1.0" />
+                <mesh filename="package://iri_wam_description/mesh/wam4_collision.stl" scale="1.0 1.0 1.0" />
 <!--                <box size="0.10 0.10 0.10"/> -->
             </geometry>

File: iri_wam_description/xacro/iri_wam_5.urdf.xacro (robot description, xacro)
@@ -14,5 +14,5 @@
             <origin xyz="0.0 0.0 0.0" rpy="0 0 0" />
             <geometry name="${prefix}_link_5_visual">
-                <mesh filename="model://iri_wam_description/mesh/wam5.stl" scale="1.0 1.0 1.0" />
+                <mesh filename="package://iri_wam_description/mesh/wam5.stl" scale="1.0 1.0 1.0" />
             </geometry>
             <material name="Grey" >
@@ -23,5 +23,5 @@
             <origin xyz="0.0 0.0 0.0" rpy="0 0 0"/>
             <geometry name="${prefix}_link_5_collision">
-                <mesh filename="model://iri_wam_description/mesh/wam5_collision.stl" scale="1.0 1.0 1.0" />
+                <mesh filename="package://iri_wam_description/mesh/wam5_collision.stl" scale="1.0 1.0 1.0" />
 <!--                <box size="0.10 0.10 0.10"/> -->
             </geometry>

File: iri_wam_description/xacro/iri_wam_6.urdf.xacro (robot description, xacro)
@@ -14,5 +14,5 @@
             <origin xyz="0.0 0.0 0.0" rpy="0 0 0" />
             <geometry name="${prefix}_link_6_visual">
-                <mesh filename="model://iri_wam_description/mesh/wam6.stl" scale="1.0 1.0 1.0" />
+                <mesh filename="package://iri_wam_description/mesh/wam6.stl" scale="1.0 1.0 1.0" />
             </geometry>
             <material name="Grey" >
@@ -23,5 +23,5 @@
             <origin xyz="0.0 0.0 0.0" rpy="0 0 0"/>
             <geometry name="${prefix}_link_6_collision">
-                <mesh filename="model://iri_wam_description/mesh/wam6_collision.stl" scale="1.0 1.0 1.0" />
+                <mesh filename="package://iri_wam_description/mesh/wam6_collision.stl" scale="1.0 1.0 1.0" />
 <!--                <box size="0.10 0.10 0.10"/> -->
             </geometry>

File: iri_wam_description/xacro/iri_wam_7.urdf.xacro (robot description, xacro)
@@ -14,5 +14,5 @@
             <origin xyz="0.0 0.0 0.0" rpy="0 0 0" />
             <geometry name="${prefix}_link_7_visual">
-                <mesh filename="model://iri_wam_description/mesh/wam7.stl" scale="1.0 1.0 1.0" />
+                <mesh filename="package://iri_wam_description/mesh/wam7.stl" scale="1.0 1.0 1.0" />
             </geometry>
             <material name="Grey" >
@@ -23,5 +23,5 @@
             <origin xyz="0.0 0.0 0.0" rpy="0 0 0"/>
             <geometry name="${prefix}_link_7_collision">
-                <mesh filename="model://iri_wam_description/mesh/wam7_collision.stl" scale="1.0 1.0 1.0" />
+                <mesh filename="package://iri_wam_description/mesh/wam7_collision.stl" scale="1.0 1.0 1.0" />
 <!--                <box size="0.10 0.10 0.10"/> -->
             </geometry>

File: iri_wam_description/xacro/iri_wam_base.urdf.xacro (robot description, xacro)
@@ -18,5 +18,5 @@
             <origin xyz="0 0 0" rpy="0 0 0" />
             <geometry>
-                <mesh filename="model://iri_wam_description/mesh/wambase.stl" scale="1.0 1.0 1.0" />
+                <mesh filename="package://iri_wam_description/mesh/wambase.stl" scale="1.0 1.0 1.0" />
             </geometry>
             <material name="Grey" >
@@ -27,5 +27,5 @@
             <origin xyz="0.0 0.0 0.0" rpy="0 0 0"/>
             <geometry>
-                <mesh filename="model://iri_wam_description/mesh/wambase_collision.stl" scale="1.0 1.0 1.0" />
+                <mesh filename="package://iri_wam_description/mesh/wambase_collision.stl" scale="1.0 1.0 1.0" />
             </geometry>
             <contact_coefficients kd="1.0" kp="1000.0" mu="0"/>

File: iri_wam_description/xacro/misc/hokuyo_laser.urdf.xacro (robot description, xacro)
@@ -18,5 +18,5 @@
             <origin xyz="0 0 0" rpy="0 0 0"/>
             <geometry>
-                <mesh filename="model://hokuyo/meshes/hokuyo.dae"/>
+                <mesh filename="package://hokuyo/meshes/hokuyo.dae"/>
             </geometry>
             <material name="Grey"/>

File: iri_wam_description/xacro/misc/kinect.urdf.xacro (robot description, xacro)
@@ -87,5 +87,5 @@
        <origin xyz="0 0 0" rpy="0 0 ${M_PI/2}"/>
         <geometry>
-         <mesh filename="model://turtlebot_description/meshes/sensors/kinect.dae"/>
+         <mesh filename="package://turtlebot_description/meshes/sensors/kinect.dae"/>
         </geometry>
       </visual>

File: iri_wam_description/xacro/misc/spoon.urdf.xacro (robot description, xacro)
@@ -12,5 +12,5 @@
        <origin xyz="0.0 -0.00 0.02" rpy="1.3 0.0 -1.1"/>
         <geometry>
-         <mesh filename="model://iri_wam_description/mesh/round_spoon/meshes/round_soup_spoon.dae"/>
+         <mesh filename="package://iri_wam_description/mesh/round_spoon/meshes/round_soup_spoon.dae"/>
         </geometry>
       </visual>
@@ -18,5 +18,5 @@
         <origin xyz="0.0 -0.0 0.02" rpy="1.3 0.0 -1.1"/>
         <geometry>
-          <mesh filename="model://iri_wam_description/mesh/round_spoon/meshes/round_soup_spoon.dae"/>
+          <mesh filename="package://iri_wam_description/mesh/round_spoon/meshes/round_soup_spoon.dae"/>
         </geometry>
       </collision>
