Commit message: Modified path to hokuyo laser

File: iri_wam_description/xacro/misc/hokuyo_laser.urdf.xacro (robot description, xacro)
@@ -18,5 +18,5 @@
             <origin xyz="0 0 0" rpy="0 0 0"/>
             <geometry>
-                <mesh filename="package://hokuyo/meshes/hokuyo.dae"/>
+                <mesh filename="package://gazebo_plugins/test/multi_robot_scenario/meshes/laser/hokuyo.dae"/>
             </geometry>
             <material name="Grey"/>
