Commit message: Updated urdfs

File: iri_wam_description/xacro/iri_wam.urdf.xacro (robot description, xacro)
@@ -22,5 +22,5 @@
        the origin block defines where the component is w.r.t its parent (in this case the parent
        is the world frame). For more, see http://www.ros.org/wiki/xacro -->
-  <property name="robot_name" value="iri_wam"/>
+  <xacro:property name="robot_name" value="iri_wam"/>
   <!-- This will attach the robot to the world link -->
   <link name="world"/>

File: iri_wam_description/xacro/iri_wam_1.urdf.xacro (robot description, xacro)
@@ -1,5 +1,5 @@
 <?xml version="1.0"?>
 <robot xmlns:xacro="http://www.ros.org/wiki/xacro">
-  <property name="M_PI" value="3.1415926535897931" />
+  <xacro:property name="M_PI" value="3.1415926535897931" />
   <xacro:macro name="wam1" params="prefix parent">
     <link name="${prefix}_link_1">
@@ -45,8 +45,8 @@
       <type>transmission_interface/SimpleTransmission</type>
       <joint name="${prefix}_joint_1">
-       <hardwareInterface>EffortJointInterface</hardwareInterface>
+       <hardwareInterface>hardware_interface/EffortJointInterface</hardwareInterface>
       </joint>
       <actuator name="motor_1">
-        <hardwareInterface>EffortJointInterface</hardwareInterface>
+        <hardwareInterface>hardware_interface/EffortJointInterface</hardwareInterface>
       	<mechanicalReduction>50</mechanicalReduction>
         <motorTorqueConstant>1</motorTorqueConstant>

File: iri_wam_description/xacro/iri_wam_2.urdf.xacro (robot description, xacro)
@@ -1,5 +1,5 @@
 <?xml version="1.0"?>
 <robot xmlns:xacro="http://www.ros.org/wiki/xacro">
-  <property name="M_PI" value="3.1415926535897931" />
+  <xacro:property name="M_PI" value="3.1415926535897931" />
   <xacro:macro name="wam2" params="prefix parent">
     <link name="${prefix}_link_2">
@@ -45,8 +45,8 @@
       <type>transmission_interface/SimpleTransmission</type>
       <joint name="${prefix}_joint_2">
-      <hardwareInterface>EffortJointInterface</hardwareInterface>
+      <hardwareInterface>hardware_interface/EffortJointInterface</hardwareInterface>
       </joint>
       <actuator name="motor_2">
-        <hardwareInterface>EffortJointInterface</hardwareInterface>
+        <hardwareInterface>hardware_interface/EffortJointInterface</hardwareInterface>
       	<mechanicalReduction>50</mechanicalReduction>
         <motorTorqueConstant>1</motorTorqueConstant>

File: iri_wam_description/xacro/iri_wam_3.urdf.xacro (robot description, xacro)
@@ -1,5 +1,5 @@
 <?xml version="1.0"?>
 <robot xmlns:xacro="http://www.ros.org/wiki/xacro">
-  <property name="M_PI" value="3.1415926535897931" />
+  <xacro:property name="M_PI" value="3.1415926535897931" />
   <xacro:macro name="wam3" params="prefix parent">
     <link name="${prefix}_link_3">
@@ -45,8 +45,8 @@
       <type>transmission_interface/SimpleTransmission</type>
       <joint name="${prefix}_joint_3">
-        <hardwareInterface>EffortJointInterface</hardwareInterface>
+        <hardwareInterface>hardware_interface/EffortJointInterface</hardwareInterface>
       </joint>
       <actuator name="motor_3">
-        <hardwareInterface>EffortJointInterface</hardwareInterface>
+        <hardwareInterface>hardware_interface/EffortJointInterface</hardwareInterface>
       	<mechanicalReduction>50</mechanicalReduction>
         <motorTorqueConstant>1</motorTorqueConstant>

File: iri_wam_description/xacro/iri_wam_4.urdf.xacro (robot description, xacro)
@@ -1,5 +1,5 @@
 <?xml version="1.0"?>
 <robot xmlns:xacro="http://www.ros.org/wiki/xacro">
-  <property name="M_PI" value="3.1415926535897931" />
+  <xacro:property name="M_PI" value="3.1415926535897931" />
   <xacro:macro name="wam4" params="prefix parent">
     <link name="${prefix}_link_4">
@@ -45,8 +45,8 @@
       <type>transmission_interface/SimpleTransmission</type>
       <joint name="${prefix}_joint_4">
-        <hardwareInterface>EffortJointInterface</hardwareInterface>
+        <hardwareInterface>hardware_interface/EffortJointInterface</hardwareInterface>
       </joint>
       <actuator name="motor_4">
-        <hardwareInterface>EffortJointInterface</hardwareInterface>
+        <hardwareInterface>hardware_interface/EffortJointInterface</hardwareInterface>
       	<mechanicalReduction>50</mechanicalReduction>
         <motorTorqueConstant>1</motorTorqueConstant>

File: iri_wam_description/xacro/iri_wam_5.urdf.xacro (robot description, xacro)
@@ -1,5 +1,5 @@
 <?xml version="1.0"?>
 <robot xmlns:xacro="http://www.ros.org/wiki/xacro">
-  <property name="M_PI" value="3.1415926535897931" />
+  <xacro:property name="M_PI" value="3.1415926535897931" />
   <xacro:macro name="wam5" params="prefix parent">
     <link name="${prefix}_link_5">
@@ -45,8 +45,8 @@
       <type>transmission_interface/SimpleTransmission</type>
       <joint name="${prefix}_joint_5">
-        <hardwareInterface>EffortJointInterface</hardwareInterface>
-</joint>
+        <hardwareInterface>hardware_interface/EffortJointInterface</hardwareInterface>
+      </joint>
       <actuator name="motor_5">
-        <hardwareInterface>EffortJointInterface</hardwareInterface>
+        <hardwareInterface>hardware_interface/EffortJointInterface</hardwareInterface>
       	<mechanicalReduction>50</mechanicalReduction>
         <motorTorqueConstant>1</motorTorqueConstant>

File: iri_wam_description/xacro/iri_wam_6.urdf.xacro (robot description, xacro)
@@ -1,5 +1,5 @@
 <?xml version="1.0"?>
 <robot xmlns:xacro="http://www.ros.org/wiki/xacro">
-  <property name="M_PI" value="3.1415926535897931" />
+  <xacro:property name="M_PI" value="3.1415926535897931" />
   <xacro:macro name="wam6" params="prefix parent">
     <link name="${prefix}_link_6">
@@ -45,8 +45,8 @@
       <type>transmission_interface/SimpleTransmission</type>
       <joint name="${prefix}_joint_6">
-        <hardwareInterface>EffortJointInterface</hardwareInterface>
-</joint>
+        <hardwareInterface>hardware_interface/EffortJointInterface</hardwareInterface>
+      </joint>
       <actuator name="motor_6">
-        <hardwareInterface>EffortJointInterface</hardwareInterface>
+        <hardwareInterface>hardware_interface/EffortJointInterface</hardwareInterface>
       	<mechanicalReduction>50</mechanicalReduction>
         <motorTorqueConstant>1</motorTorqueConstant>

File: iri_wam_description/xacro/iri_wam_7.urdf.xacro (robot description, xacro)
@@ -1,5 +1,5 @@
 <?xml version="1.0"?>
 <robot xmlns:xacro="http://www.ros.org/wiki/xacro">
-  <property name="M_PI" value="3.1415926535897931" />
+  <xacro:property name="M_PI" value="3.1415926535897931" />
   <xacro:macro name="wam7" params="prefix parent">
     <link name="${prefix}_link_7">
@@ -45,8 +45,8 @@
       <type>transmission_interface/SimpleTransmission</type>
       <joint name="${prefix}_joint_7">
-        <hardwareInterface>EffortJointInterface</hardwareInterface>
-</joint>
+        <hardwareInterface>hardware_interface/EffortJointInterface</hardwareInterface>
+      </joint>
       <actuator name="motor_7">
-        <hardwareInterface>EffortJointInterface</hardwareInterface>
+        <hardwareInterface>hardware_interface/EffortJointInterface</hardwareInterface>
       	<mechanicalReduction>50</mechanicalReduction>
         <motorTorqueConstant>1</motorTorqueConstant>

File: iri_wam_description/xacro/iri_wam_base.urdf.xacro (robot description, xacro)
@@ -1,9 +1,9 @@
 <?xml version="1.0"?>
 <robot xmlns:xacro="http://ros.org/wiki/xacro">
-  <property name="M_PI" value="3.1415926535897931" />
-  <property name="base_mass" value="20"/>
-  <property name="base_cg_x" value="0.0"/>
-  <property name="base_cg_y" value="0.0"/>
-  <property name="base_cg_z" value="0.0"/>
+  <xacro:property name="M_PI" value="3.1415926535897931" />
+  <xacro:property name="base_mass" value="20"/>
+  <xacro:property name="base_cg_x" value="0.0"/>
+  <xacro:property name="base_cg_y" value="0.0"/>
+  <xacro:property name="base_cg_z" value="0.0"/>
   <xacro:macro name="wambase" params="prefix">
     <link name="${prefix}_link_base">

File: iri_wam_description/xacro/iri_wam_tcp.urdf.xacro (robot description, xacro)
@@ -1,5 +1,5 @@
 <?xml version="1.0"?>
 <robot xmlns:xacro="http://www.ros.org/wiki/xacro">
-  <property name="M_PI" value="3.1415926535897931" />
+  <xacro:property name="M_PI" value="3.1415926535897931" />
   <xacro:macro name="wamtcp" params="prefix parent">
     <link name="${prefix}_link_tcp" />

File: iri_wam_description/xacro/misc/cylinder.urdf.xacro (robot description, xacro)
@@ -1,12 +1,12 @@
 <?xml version="1.0"?>
 <robot name="cylinder" xmlns:xacro="http://ros.org/wiki/xacro">
-  <property name="object_1_x" value="0.0" />
-  <property name="object_1_y" value="0.0" />
-  <property name="object_1_height"      value="1.2" />
-  <property name="object_1_radius"      value="0.02" />
-  <property name="object_1_base_height" value="0.02" />
-  <property name="object_1_base_width"  value="0.15" />
-  <property name="object_1_mass"        value="0.2" />
-  <property name="object_1_mu"          value="500.0" />
+  <xacro:property name="object_1_x" value="0.0" />
+  <xacro:property name="object_1_y" value="0.0" />
+  <xacro:property name="object_1_height"      value="1.2" />
+  <xacro:property name="object_1_radius"      value="0.02" />
+  <xacro:property name="object_1_base_height" value="0.02" />
+  <xacro:property name="object_1_base_width"  value="0.15" />
+  <xacro:property name="object_1_mass"        value="0.2" />
+  <xacro:property name="object_1_mu"          value="500.0" />
   <link name="cylinder">
     <inertial>

File: iri_wam_description/xacro/misc/cylinder_object.urdf.xacro (robot description, xacro)
@@ -13,14 +13,14 @@
        xmlns:controller="http://playerstage.sourceforge.net/gazebo/xmlschema/#controller"
        xmlns:physics="http://playerstage.sourceforge.net/gazebo/xmlschema/#physics">
-  <property name="table_z" value="0.0" />
-  <property name="table_height" value="0.55" />
-  <property name="object_1_x" value="0.0" />
-  <property name="object_1_y" value="0.0" />
-  <property name="object_1_height"      value="1.2" />
-  <property name="object_1_radius"      value="0.02" />
-  <property name="object_1_base_height" value="0.02" />
-  <property name="object_1_base_width"  value="0.15" />
-  <property name="object_1_mass"        value="0.2" />
-  <property name="object_1_mu"          value="500.0" />
+  <xacro:property name="table_z" value="0.0" />
+  <xacro:property name="table_height" value="0.55" />
+  <xacro:property name="object_1_x" value="0.0" />
+  <xacro:property name="object_1_y" value="0.0" />
+  <xacro:property name="object_1_height"      value="1.2" />
+  <xacro:property name="object_1_radius"      value="0.02" />
+  <xacro:property name="object_1_base_height" value="0.02" />
+  <xacro:property name="object_1_base_width"  value="0.15" />
+  <xacro:property name="object_1_mass"        value="0.2" />
+  <xacro:property name="object_1_mu"          value="500.0" />
   <joint name="object_1_joint" type="fixed" >
     <parent link="object_1_base_link" />

File: iri_wam_description/xacro/misc/generic_camera.urdf.xacro (robot description, xacro)
@@ -5,9 +5,9 @@
   xmlns:xacro="http://ros.org/wiki/xacro"
   >
-    <property name="M_PI" value="3.1415926535897931" />
+    <xacro:property name="M_PI" value="3.1415926535897931" />
     <xacro:macro name="generic_camera" params="name parent  ros_topic cam_info_topic update_rate res_x res_y image_format hfov">
       <joint name="${name}_joint" type="fixed">
         <origin xyz="0 0 0.09" rpy="0.0 ${-M_PI/2} 0.0" />
-        <insert_block name="origin" />
+        <xacro:insert_block name="origin" />
         <parent link="${parent}"/>
         <child link="${name}_link"/>

File: iri_wam_description/xacro/misc/iri_wam.gazebo.xacro (robot description, xacro)
@@ -4,5 +4,5 @@
        xmlns:interface="http://playerstage.sourceforge.net/gazebo/xmlschema/#interface"
        name="iri_wam">
-  <include filename="$(find iri_wam_description)/xacro/wam.urdf.xacro" />
+  <xacro:include filename="$(find iri_wam_description)/xacro/wam.urdf.xacro" />
   <gazebo>
 	<controller:gazebo_ros_controller_manager name="gazebo_ros_controller_manager" plugin="libgazebo_ros_controller_manager.so">

File: iri_wam_description/xacro/misc/kinect.urdf.xacro (robot description, xacro)
@@ -1,11 +1,11 @@
 <?xml version="1.0" ?>
 <robot xmlns:xacro="http://ros.org/wiki/xacro" >
-  <property name="M_PI" value="3.1415926535897931" />
-	<property name="cam_px" value="-0.1" />
-	<property name="cam_py" value="-0.0125" />
-	<property name="cam_pz" value=" 0.08" />
-	<property name="cam_or" value="0" />
-	<property name="cam_op" value="-${M_PI/2}" />
-	<property name="cam_oy" value="0" />
+  <xacro:property name="M_PI" value="3.1415926535897931" />
+	<xacro:property name="cam_px" value="-0.1" />
+	<xacro:property name="cam_py" value="-0.0125" />
+	<xacro:property name="cam_pz" value=" 0.08" />
+	<xacro:property name="cam_or" value="0" />
+	<xacro:property name="cam_op" value="-${M_PI/2}" />
+	<xacro:property name="cam_oy" value="0" />
   <xacro:macro name="kinect" params="prefix parent">
     <gazebo reference="camera_link">

File: iri_wam_description/xacro/misc/light_sensor.urdf.xacro (robot description, xacro)
@@ -4,9 +4,9 @@
 xmlns:interface="http://playerstage.sourceforge.net/gazebo/xmlschema/#interface"
   xmlns:xacro="http://ros.org/wiki/xacro" >
-    <property name="M_PI" value="3.1415926535897931" />
+    <xacro:property name="M_PI" value="3.1415926535897931" />
     <xacro:macro name="light_sensor" params="name prefix parent *origin ros_topic cam_info_topic update_rate res_x res_y image_format hfov">
       <joint name="${name}_joint" type="fixed">
         <origin xyz="0 0 0.09" rpy="0.0 ${-M_PI/2} 0.0" />
-        <insert_block name="origin" />
+        <xacro:insert_block name="origin" />
         <parent link="${parent}"/>
         <child link="${name}_link"/>

File: iri_wam_description/xacro/misc/spoon.urdf.xacro (robot description, xacro)
@@ -1,5 +1,5 @@
 <?xml version="1.0" ?>
 <robot xmlns:xacro="http://ros.org/wiki/xacro" >
-  <property name="M_PI" value="3.1415926535897931" />
+  <xacro:property name="M_PI" value="3.1415926535897931" />
   <xacro:macro name="spoon" params="prefix parent">
     <joint name="spoon_joint" type="fixed">

File: iri_wam_description/xacro/misc/table.urdf.xacro (robot description, xacro)
@@ -1,12 +1,12 @@
 <?xml version="1.0"?>
 <robot name="table" xmlns:xacro="http://www.ros.org/wiki/xacro">
-  <property name="table_height" value="0.9" />
-  <property name="table_width" value="1.2" />
-  <property name="table_depth" value="0.5" />
-  <property name="table_x" value="0.0" />
-  <property name="table_y" value="0.0" />
-  <property name="table_z" value="0.0" />
-  <property name="table_top_thickness" value="0.05"/>
-  <property name="M_PI" value="3.1415926535897931" />
+  <xacro:property name="table_height" value="0.9" />
+  <xacro:property name="table_width" value="1.2" />
+  <xacro:property name="table_depth" value="0.5" />
+  <xacro:property name="table_x" value="0.0" />
+  <xacro:property name="table_y" value="0.0" />
+  <xacro:property name="table_z" value="0.0" />
+  <xacro:property name="table_top_thickness" value="0.05"/>
+  <xacro:property name="M_PI" value="3.1415926535897931" />
   <link name ="world" />
   <link name="leg_1">

File: iri_wam_description/xacro/misc/vertical_stick.urdf.xacro (robot description, xacro)
@@ -13,14 +13,14 @@
        xmlns:controller="http://playerstage.sourceforge.net/gazebo/xmlschema/#controller"
        xmlns:physics="http://playerstage.sourceforge.net/gazebo/xmlschema/#physics">
-  <property name="vertical_stick_z" value="0.0" />
-  <property name="vertical_stick_height" value="0.55" />
-  <property name="vertical_stick_x" value="0.0" />
-  <property name="vertical_stick_y" value="0.0" />
-  <property name="vertical_stick_height"      value="1.2" />
-  <property name="vertical_stick_radius"      value="0.02" />
-  <property name="vertical_stick_base_height" value="0.02" />
-  <property name="vertical_stick_base_width"  value="0.15" />
-  <property name="vertical_stick_mass"        value="0.2" />
-  <property name="vertical_stick_mu"          value="500.0" />
+  <xacro:property name="vertical_stick_z" value="0.0" />
+  <xacro:property name="vertical_stick_height" value="0.55" />
+  <xacro:property name="vertical_stick_x" value="0.0" />
+  <xacro:property name="vertical_stick_y" value="0.0" />
+  <xacro:property name="vertical_stick_height"      value="1.2" />
+  <xacro:property name="vertical_stick_radius"      value="0.02" />
+  <xacro:property name="vertical_stick_base_height" value="0.02" />
+  <xacro:property name="vertical_stick_base_width"  value="0.15" />
+  <xacro:property name="vertical_stick_mass"        value="0.2" />
+  <xacro:property name="vertical_stick_mu"          value="500.0" />
   <joint name="vertical_stick_joint" type="fixed" >
     <parent link="vertical_stick_base_link" />

File: iri_wam_description/xacro/misc/wam_with_camera.urdf.xacro (robot description, xacro)
@@ -6,17 +6,17 @@
        name="iri_wam">
   <!-- LINKS   -->
-<!--  <include filename="$(find iri_wam_description)/xacro/wambase.urdf.xacro" />
+<!--  <xacro:include filename="$(find iri_wam_description)/xacro/wambase.urdf.xacro" />
 -->
-  <include filename="$(find iri_wam_description)/xacro/wam0.urdf.xacro" />
-  <include filename="$(find iri_wam_description)/xacro/wam1.urdf.xacro" />
-  <include filename="$(find iri_wam_description)/xacro/wam2.urdf.xacro" />
-  <include filename="$(find iri_wam_description)/xacro/wam3.urdf.xacro" />
-  <include filename="$(find iri_wam_description)/xacro/wam4.urdf.xacro" />
-  <include filename="$(find iri_wam_description)/xacro/wam5.urdf.xacro" />
-  <include filename="$(find iri_wam_description)/xacro/wam6.urdf.xacro" />
-  <include filename="$(find iri_wam_description)/xacro/wam7.urdf.xacro" />
-  <include filename="$(find iri_wam_description)/xacro/wamtcp.urdf.xacro" />
+  <xacro:include filename="$(find iri_wam_description)/xacro/wam0.urdf.xacro" />
+  <xacro:include filename="$(find iri_wam_description)/xacro/wam1.urdf.xacro" />
+  <xacro:include filename="$(find iri_wam_description)/xacro/wam2.urdf.xacro" />
+  <xacro:include filename="$(find iri_wam_description)/xacro/wam3.urdf.xacro" />
+  <xacro:include filename="$(find iri_wam_description)/xacro/wam4.urdf.xacro" />
+  <xacro:include filename="$(find iri_wam_description)/xacro/wam5.urdf.xacro" />
+  <xacro:include filename="$(find iri_wam_description)/xacro/wam6.urdf.xacro" />
+  <xacro:include filename="$(find iri_wam_description)/xacro/wam7.urdf.xacro" />
+  <xacro:include filename="$(find iri_wam_description)/xacro/wamtcp.urdf.xacro" />
   <!-- Forward facing camera -->
-  <include filename="$(find iri_wam_description)/xacro/misc/generic_camera.urdf.xacro" />
+  <xacro:include filename="$(find iri_wam_description)/xacro/misc/generic_camera.urdf.xacro" />
 <!--
   <xacro:wambase>
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